File: PCB/KiCad/tvbgone_kit_v2.0/tvbgone_kit_v2.0.kicad_pcb (KiCad board)
At the start: 2 copper layers, 59.9 x 49.3 mm, 24 parts, among them Q1 IRLU024NPBF

Commit message: Changed resistor values to prevent LED burnout on high current supply. Cleaned up the built board look by moving references inside footprints. Reduced font size from 1 -> 0.75 on some components to fit references. Changed B1 to Battery for more straight-forward build process.
Parts:
- R1, R2, R3, R4: value 0.47 -> 120
- R5, R6: moved to F.Cu
- turned R5 to 180 degrees
- turned R6 to 180 degrees
- renumbered B1 to Battery
Other:
- board text added: "120"
- board text removed: "0.47"

Commit message: draft r2: IR LEDs on GPIO4
* Changed IR LEDs from GPIO2 to GPIO4 (since GPIO2 goes High during bootloader programming, burning out the IR LEDs).
* Fixed label reversal of R5 and R6
* Cleaned up some silk screen
* Added IR Receiver for learning IR codes (but firmware not implemented).
Parts:
- added U1: TSOP38238, OptoDevice:Vishay_MINICAST-3Pin, F.Cu at (118.0, 88.3)
- R5, R6: moved to B.Cu
- turned R5 to 0 degrees
- turned R6 to 0 degrees
- renumbered Battery to B1
Connections:
- MOD1 pad 11: Net-(MOD1-GPIO2) -> unconnected-(MOD1-GPIO2-Pad11)
- MOD1 pad 12: unconnected-(MOD1-GPIO3-Pad12) -> Net-(MOD1-GPIO3)
- MOD1 pad 13: unconnected-(MOD1-GPIO4-Pad13) -> Net-(MOD1-GPIO4)
- R5 pad P$1: Net-(MOD1-GPIO2) -> Net-(MOD1-GPIO4)
Routing:
- net Net-(MOD1-GPIO4): track 0.00 -> 63.1 mm
- net Net-(MOD1-GPIO2): track 59.8 -> 0.00 mm
- net Net-(MOD1-GPIO3): track 0.00 -> 46.7 mm
- net GND: track 189.9 -> 196.7 mm
- net +4.5V: track 76.0 -> 80.6 mm
Other:
- board text added: "+"
- board text added: "-"
- board text added: "3.3"
- board text added: "TSOP38238"
- board text added: "kit V2.0 r2"
- board text removed: "120"
- board text removed: "kit V2.0 r1"
