File: PCB/KiCad/tvbgone_kit_v2.0/tvbgone_kit_v2.0.kicad_sch (KiCad schematic)
At the start: 18 parts, among them Q1 IRLU024NPBF

Commit message: Changed resistor values to prevent LED burnout on high current supply. Cleaned up the built board look by moving references inside footprints. Reduced font size from 1 -> 0.75 on some components to fit references. Changed B1 to Battery for more straight-forward build process.
Parts:
- R1, R2, R3, R4: value 0.47 -> 120
Changed lines of the file:
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@@
 			)
 		)
-		(property "Value" "0.47"
+		(property "Value" "120"
 			(at 167.132 87.63 90)
 			(effects
@@
 			)
 		)
-		(property "Value" "0.47"
+		(property "Value" "120"
 			(at 179.832 87.63 90)
 			(effects
@@
 			)
 		)
-		(property "Value" "0.47"
+		(property "Value" "120"
 			(at 192.532 87.63 90)
 			(effects
@@
 			)
 		)
-		(property "Value" "0.47"
+		(property "Value" "120"
 			(at 205.232 87.63 90)
 			(effects

Commit message: draft r2: IR LEDs on GPIO4
* Changed IR LEDs from GPIO2 to GPIO4 (since GPIO2 goes High during bootloader programming, burning out the IR LEDs).
* Fixed label reversal of R5 and R6
* Cleaned up some silk screen
* Added IR Receiver for learning IR codes (but firmware not implemented).
Parts:
- added U1: TSOP38238, OptoDevice:Vishay_MINICAST-3Pin, symbol Interface_Optical:TSOP382xx
Connections:
- net +4.5V: now also U1.3 (Vs)
- net GND: now also U1.2 (GND)
- net at R5.P$1: now also MOD1.13 (GPIO4); no longer MOD1.11 (GPIO2)
- net at MOD1.12 (GPIO3): now also U1.1 (OUT)
- no-connect marks 13 -> 12
Other:
- title: TV-B-Gone kit V2 -- preliminary PCB -> TV-B-Gone kit V2 -- preliminary PCB r2
