File: PCB/KiCad/tvbgone_kit_v2.0/tvbgone_kit_v2.0.kicad_sch (KiCad schematic)
At the start: 19 parts, among them Q1 IRLU024NPBF, U1 TSOP38238

Commit message: new IR LED resistors, updated BOM & assembly
* After testing, R1-R4 were reduced to 1 Ohm to maximize range of IR LEDs.
* Updated BOM.
* Put Gerber files in their own subdirectory.
Parts:
- R1, R2, R3, R4: value 120 -> 1; Part # KOA Speer -- MOSX1/2CT52RR47J -> Stackpole -- CFM12JT1R00
Other:
- note added: "Other options for Q1: Doingter DOU90N02 (from LCSC) NCE NCE3080IA (from LCSC)"
Changed lines of the file:
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@@
 	(title_block
 		(title "TV-B-Gone kit V2 -- preliminary PCB r2")
-		(date "2026-04-30")
+		(date "2026-05-14")
 		(rev "r2")
 		(company "Cornfield Electronics")
@@
 	(text "Thermal pad"
 		(exclude_from_sim no)
-		(at 182.372 108.204 0)
+		(at 196.85 109.474 0)
 		(effects
 			(font
@@
 		)
 	)
+	(text "Other options for Q1:\n   Doingter DOU90N02 (from LCSC)\n   NCE NCE3080IA  (from LCSC)"
+		(exclude_from_sim no)
+		(at 184.912 125.984 0)
+		(effects
+			(font
+				(size 1.27 1.27)
+			)
+			(justify left)
+		)
+	)
 	(junction
 		(at 170.18 118.11)
@@
 			)
 		)
-		(property "Value" "120"
-			(at 167.132 87.63 90)
+		(property "Value" "1"
+			(at 165.862 87.63 90)
 			(show_name no)
 			(do_not_autoplace no)
@@
 			)
 		)
-		(property "Datasheet" "https://www.koaspeer.com/pdfs/MOS.pdf"
+		(property "Datasheet" "https://www.seielect.com/catalog/SEI-CF_CFM.pdf"
 			(at 163.83 87.63 0)
 			(hide yes)
@@
 			)
 		)
-		(property "Description" "0.47 Ohm, 1/2W, 5%"
+		(property "Description" "1 Ohm, 1/2W, 5%"
 			(at 168.91 87.63 0)
 			(hide yes)
@@
 			)
 		)
-		(property "Part #" "KOA Speer -- MOSX1/2CT52RR47J "
+		(property "Part #" "Stackpole -- CFM12JT1R00"
 			(at 163.83 87.63 0)
 			(hide yes)
@@
 			)
 		)
-		(property "Value" "120"
-			(at 179.832 87.63 90)
+		(property "Value" "1"
+			(at 178.816 87.63 90)
 			(show_name no)
 			(do_not_autoplace no)
@@
 			)
 		)
-		(property "Datasheet" "https://www.koaspeer.com/pdfs/MOS.pdf"
+		(property "Datasheet" "https://www.seielect.com/catalog/SEI-CF_CFM.pdf"
 			(at 176.53 87.63 0)
 			(hide yes)
@@
 			)
 		)
-		(property "Description" "0.47 Ohm, 1/2W, 5%"
+		(property "Description" "1 Ohm, 1/2W, 5%"
 			(at 181.61 87.63 0)
 			(hide yes)
@@
 			)
 		)
-		(property "Part #" "KOA Speer -- MOSX1/2CT52RR47J "
+		(property "Part #" "Stackpole -- CFM12JT1R00"
 			(at 176.53 87.63 0)
 			(hide yes)
@@
 			)
 		)
-		(property "Value" "120"
-			(at 192.532 87.63 90)
+		(property "Value" "1"
+			(at 191.516 87.63 90)
 			(show_name no)
 			(do_not_autoplace no)
@@
 			)
 		)
-		(property "Datasheet" "https://www.koaspeer.com/pdfs/MOS.pdf"
+		(property "Datasheet" "https://www.seielect.com/catalog/SEI-CF_CFM.pdf"
 			(at 189.23 87.63 0)
 			(hide yes)
@@
 			)
 		)
-		(property "Description" "0.47 Ohm, 1/2W, 5%"
+		(property "Description" "1 Ohm, 1/2W, 5%"
 			(at 194.31 87.63 0)
 			(hide yes)
@@
 			)
 		)
-		(property "Part #" "KOA Speer -- MOSX1/2CT52RR47J "
+		(property "Part #" "Stackpole -- CFM12JT1R00"
 			(at 189.23 87.63 0)
 			(hide yes)
@@
 			)
 		)
-		(property "Value" "120"
-			(at 205.232 87.63 90)
+		(property "Value" "1"
+			(at 204.216 87.63 90)
 			(show_name no)
 			(do_not_autoplace no)
@@
 			)
 		)
-		(property "Datasheet" "https://www.koaspeer.com/pdfs/MOS.pdf"
+		(property "Datasheet" "https://www.seielect.com/catalog/SEI-CF_CFM.pdf"
 			(at 201.93 87.63 0)
 			(hide yes)
@@
 			)
 		)
-		(property "Description" "0.47 Ohm, 1/2W, 5%"
+		(property "Description" "1 Ohm, 1/2W, 5%"
 			(at 207.01 87.63 0)
 			(hide yes)
@@
 			)
 		)
-		(property "Part #" "KOA Speer -- MOSX1/2CT52RR47J "
+		(property "Part #" "Stackpole -- CFM12JT1R00"
 			(at 201.93 87.63 0)
 			(hide yes)

Commit message: Change C2 to 0.1" lead-spacing
Change C2 to 0.1" lead-spacing
C2 part number changed from Panasonic ECE-A0JKA331Q to Panasonic ECE-A0JKA331
Parts:
- C2: Part # Panasonic -- ECE-A0JKA331Q -> Panasonic -- ECE-A0JKA331
Other:
- title: TV-B-Gone kit V2 -- preliminary PCB r2 -> TV-B-Gone kit V2 -- preliminary PCB r3
Changed lines of the file:
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@@
 	(paper "A4")
 	(title_block
-		(title "TV-B-Gone kit V2 -- preliminary PCB r2")
-		(date "2026-05-14")
-		(rev "r2")
+		(title "TV-B-Gone kit V2 -- preliminary PCB r3")
+		(date "2026-06-24")
+		(rev "r3")
 		(company "Cornfield Electronics")
 		(comment 1 "Mitch Altman")
@@
 			)
 		)
-		(property "Part #" "Panasonic -- ECE-A0JKA331Q"
+		(property "Part #" "Panasonic -- ECE-A0JKA331"
 			(at 104.14 78.74 0)
 			(hide yes)
